Commit message: fixed gazebo ur moveit launch

File: Task1/ur_description/urdf/ur_macro.xacro (robot description, xacro)
@@ -375,10 +375,10 @@
     </joint>
     <!-- newly added by me -->
-    <joint name="${tf_prefix}ee_fixed_joint" type="fixed">
+    <!-- <joint name="${tf_prefix}ee_fixed_joint" type="fixed">
       <parent link="${tf_prefix}wrist_3_link" />
       <child link = "${tf_prefix}ee_link" />
       <origin xyz="0.0 0.0 0.0" rpy="0.0 0.0 0.0" />
-    </joint>
-    <link name="${tf_prefix}ee_link">
+    </joint> -->
+    <!-- <link name="${tf_prefix}ee_link">
     <visual>
       <geometry>
@@ -398,5 +398,5 @@
       <inertia ixx="0.4" ixy="0.0" ixz="0.0" iyy="0.4" iyz="0.0" izz="0.2"/>
     </inertial>
-    </link>
+    </link> -->
     <!-- End of newly added my me      -->
   </xacro:macro>

Commit message: new commits in original repo

File: Task1/ur_description/urdf/ur_macro.xacro (robot description, xacro)
@@ -375,10 +375,10 @@
     </joint>
     <!-- newly added by me -->
-    <!-- <joint name="${tf_prefix}ee_fixed_joint" type="fixed">
+    <joint name="${tf_prefix}ee_fixed_joint" type="fixed">
       <parent link="${tf_prefix}wrist_3_link" />
       <child link = "${tf_prefix}ee_link" />
       <origin xyz="0.0 0.0 0.0" rpy="0.0 0.0 0.0" />
-    </joint> -->
-    <!-- <link name="${tf_prefix}ee_link">
+    </joint>
+    <link name="${tf_prefix}ee_link">
     <visual>
       <geometry>
@@ -398,5 +398,5 @@
       <inertia ixx="0.4" ixy="0.0" ixz="0.0" iyy="0.4" iyz="0.0" izz="0.2"/>
     </inertial>
-    </link> -->
+    </link>
     <!-- End of newly added my me      -->
   </xacro:macro>

File: Task1/ur_moveit_config/srdf/ur_macro.srdf.xacro (robot description, xacro)
@@ -53,4 +53,5 @@
     <disable_collisions link1="${prefix}wrist_1_link" link2="${prefix}wrist_3_link" reason="Never" />
     <disable_collisions link1="${prefix}wrist_2_link" link2="${prefix}wrist_3_link" reason="Adjacent" />
+    <disable_collisions link1="${prefix}ee_link" link2="${prefix}wrist_3_link" reason="Adjacent" />
   </xacro:macro>
 </robot>
